File: Blinker_01.brd (EAGLE design)
At the start: 88.9 x 69.5 mm, 21 parts, among them IC1 ILQ620, X3 MSTBA6, X4 MSTBA5

Commit message: Arbeiten SW & SW zum 24.03.2020
Parts:
- added D1: THT3MM, LED:THT3MM
- added R4: 2,2k, R-C:R-10
- added U$34: TP_10", SUPPLY:TP_10
- R1, R2, R3: value (none) -> 2,2k
Connections:
- new net +5V: R4.2, U$34.P$1
- new net N$18: D1.A, R4.1
- net N$2: now also D1.K
Changed lines of the file:
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@@
 <element name="U$7" library="SUPPLY" package="TP_10" value="TP_10&quot;" x="82.55" y="53.34" rot="R180"/>
 <element name="U$8" library="SUPPLY" package="TP_10" value="TP_10&quot;" x="54.61" y="53.34" rot="R180"/>
-<element name="R1" library="R-C" package="R-10" value="" x="20.32" y="52.07"/>
-<element name="R2" library="R-C" package="R-10" value="" x="20.32" y="46.99"/>
-<element name="R3" library="R-C" package="R-10" value="" x="20.32" y="41.91"/>
+<element name="R1" library="R-C" package="R-10" value="2,2k" x="20.32" y="52.07"/>
+<element name="R2" library="R-C" package="R-10" value="2,2k" x="20.32" y="46.99"/>
+<element name="R3" library="R-C" package="R-10" value="2,2k" x="20.32" y="41.91"/>
 <element name="U$9" library="SPEZIAL" package="LDD-H" value="LDD-H" x="46.99" y="19.05" rot="R270"/>
 <element name="U$10" library="SPEZIAL" package="LDD-H" value="LDD-H" x="24.13" y="19.05" rot="R270"/>
@@
 <element name="U$33" library="SUPPLY" package="TP_10" value="TP_10&quot;" x="19.05" y="36.83"/>
 <element name="IC1" library="optocoupler" package="DIL16" value="ILQ620" x="35.56" y="49.53" rot="R270"/>
+<element name="R4" library="R-C" package="R-10" value="2,2k" x="16.51" y="60.96"/>
+<element name="D1" library="LED" package="THT3MM" value="THT3MM" x="26.67" y="59.69" rot="R90">
+<attribute name="MWNUMBER" value="" x="26.67" y="59.69" size="1.778" layer="27" rot="R90" display="off"/>
+</element>
+<element name="U$34" library="SUPPLY" package="TP_10" value="TP_10&quot;" x="66.04" y="58.42"/>
 </elements>
 <signals>
@@
 <contactref element="U$4" pad="P$1"/>
 <contactref element="IC1" pad="16"/>
+<contactref element="D1" pad="K"/>
 <wire x1="39.37" y1="58.42" x2="80.01" y2="38.1" width="0" layer="19" extent="1-1"/>
+<wire x1="26.67" y1="60.96" x2="39.37" y2="58.42" width="0" layer="19" extent="1-1"/>
 </signal>
 <signal name="N$4">
@@
 <wire x1="31.75" y1="43.18" x2="19.05" y2="36.83" width="0" layer="19" extent="1-1"/>
 </signal>
+<signal name="N$18">
+<contactref element="D1" pad="A"/>
+<contactref element="R4" pad="1"/>
+<wire x1="11.43" y1="60.96" x2="26.67" y2="58.42" width="0" layer="19" extent="1-1"/>
+</signal>
+<signal name="+5V">
+<contactref element="U$34" pad="P$1"/>
+<contactref element="R4" pad="2"/>
+<wire x1="21.59" y1="60.96" x2="66.04" y2="58.42" width="0" layer="19" extent="1-1"/>
+</signal>
 </signals>
