File: Blinker_01.sch (EAGLE design)
At the start: 21 parts, among them IC1 ILQ620, X3 MSTBA6, X4 MSTBA5

Commit message: Arbeiten SW & SW zum 24.03.2020
Parts:
- added D1: THT3MM, LED:THT3MM
- added R4: 2,2k, R-C:RESEU-10
- added U$34: TP_10", SUPPLY:TP_10"
- R1, R2, R3: value (none) -> 2,2k
Connections:
- new net +5V: R4.2, U$34.TP_13
- new net N$18: D1.P1A, R4.1
- net N$2: now also D1.P2K
Changed lines of the file:
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@@
 <setting verticaltext="up"/>
 </settings>
-<grid distance="0.05" unitdist="inch" unit="inch" style="lines" multiple="1" display="no" altdistance="0.01" altunitdist="inch" altunit="inch"/>
+<grid distance="0.1" unitdist="inch" unit="inch" style="lines" multiple="1" display="no" altdistance="0.01" altunitdist="inch" altunit="inch"/>
 <layers>
 <layer number="1" name="Top" color="4" fill="1" visible="no" active="no"/>
@@
 <part name="U$7" library="SUPPLY" deviceset="TP_10" device="&quot;"/>
 <part name="U$8" library="SUPPLY" deviceset="TP_10" device="&quot;"/>
-<part name="R1" library="R-C" deviceset="RESEU-10" device=""/>
-<part name="R2" library="R-C" deviceset="RESEU-10" device=""/>
-<part name="R3" library="R-C" deviceset="RESEU-10" device=""/>
+<part name="R1" library="R-C" deviceset="RESEU-10" device="" value="2,2k"/>
+<part name="R2" library="R-C" deviceset="RESEU-10" device="" value="2,2k"/>
+<part name="R3" library="R-C" deviceset="RESEU-10" device="" value="2,2k"/>
 <part name="U$11" library="SUPPLY" deviceset="GND" device=""/>
 <part name="U$12" library="SUPPLY" deviceset="GND" device=""/>
@@
 <part name="U$33" library="SUPPLY" deviceset="TP_10" device="&quot;"/>
 <part name="IC1" library="optocoupler" deviceset="ILQ620" device=""/>
+<part name="R4" library="R-C" deviceset="RESEU-10" device="" value="2,2k"/>
+<part name="D1" library="LED" deviceset="THT3MM" device=""/>
+<part name="U$34" library="SUPPLY" deviceset="TP_10" device="&quot;"/>
+<part name="U$35" library="SUPPLY" deviceset="+5V" device=""/>
+<part name="U$36" library="SUPPLY" deviceset="+5V" device=""/>
 </parts>
 <sheets>
@@
 <instance part="IC1" gate="C" x="91.44" y="73.66"/>
 <instance part="IC1" gate="D" x="91.44" y="50.8"/>
+<instance part="R4" gate="1" x="106.68" y="132.08" rot="R90"/>
+<instance part="D1" gate="G$1" x="106.68" y="121.92" rot="R270"/>
+<instance part="U$34" gate="G$1" x="134.62" y="144.78" rot="R180"/>
+<instance part="U$35" gate="1" x="134.62" y="147.32" rot="R180"/>
+<instance part="U$36" gate="1" x="106.68" y="137.16" rot="R180"/>
 </instances>
 <busses>
@@
 <segment>
 <pinref part="U$4" gate="G$1" pin="TP_13"/>
-<wire x1="104.14" y1="114.3" x2="127" y2="114.3" width="0.1524" layer="91"/>
+<wire x1="104.14" y1="114.3" x2="106.68" y2="114.3" width="0.1524" layer="91"/>
 <pinref part="IC1" gate="A" pin="C"/>
+<pinref part="D1" gate="G$1" pin="P2K"/>
+<wire x1="106.68" y1="114.3" x2="127" y2="114.3" width="0.1524" layer="91"/>
+<junction x="106.68" y="114.3"/>
 </segment>
 </net>
@@
 </segment>
 </net>
+<net name="N$18" class="0">
+<segment>
+<pinref part="D1" gate="G$1" pin="P1A"/>
+<pinref part="R4" gate="1" pin="1"/>
+</segment>
+</net>
+<net name="+5V" class="0">
+<segment>
+<pinref part="U$34" gate="G$1" pin="TP_13"/>
+<pinref part="U$35" gate="1" pin="+5V"/>
+</segment>
+<segment>
+<pinref part="R4" gate="1" pin="2"/>
+<pinref part="U$36" gate="1" pin="+5V"/>
+</segment>
+</net>
