File: Blinker_02.brd (EAGLE design)
At the start: 80 x 68.2 mm, 27 parts, among them IC1 ILQ620, X1 MSTBA12

Commit message: Platinendesign
Parts:
- moved D3 34.4 mm to (63.5, 40.6)
- moved D2 19.2 mm to (55.9, 40.6)
- moved U$29 15.2 mm to (68.6, 63.5)
- moved R4 10.2 mm to (17.8, 36.8), turned to 180 degrees
- moved R6 10.2 mm to (17.8, 47.0), turned to 180 degrees
- moved U$30 10.2 mm to (71.1, 63.5)
- moved D1 4.58 mm to (48.3, 40.6)
- moved U$28 2.54 mm to (61.0, 63.5)
- turned R5 to 180 degrees
Connections:
- net GND: now also X1.4
- net N$18: now also D3.A; no longer D1.A
- net N$2: now also D3.K
- net N$20: now also D1.A; no longer D3.A
- net N$3: now also D2.K
- net N$5: now also D1.K
Routing:
- net +12V: track 137.6 -> 110.5 mm
- net N$14: track 57.2 -> 79.7 mm
- net GND: track 182.2 -> 164.9 mm
- net N$13: track 40.9 -> 55.3 mm
- net N$5: track 18.1 -> 32.4 mm
- net N$20: track 18.6 -> 32.1 mm
- net N$2: track 26.3 -> 39.6 mm
- net N$19: track 27.0 -> 38.0 mm
- net N$15: track 48.6 -> 38.4 mm
- net +5V: track 37.1 -> 47.3 mm
- net N$3: track 21.7 -> 30.6 mm
- net N$18: track 37.4 -> 43.8 mm
- net N$11: track 75.0 -> 73.5 mm
- net N$12: track 91.6 -> 93.1 mm
