File: Blinker_02.sch (EAGLE design)
At the start: 27 parts, among them IC1 ILQ620, X1 MSTBA12

Commit message: Platinendesign
Connections:
- net GND: now also X1-4.1
- net N$18: now also D3.P1A; no longer D1.P1A
- net N$2: now also D3.P2K
- net N$20: now also D1.P1A; no longer D3.P1A
- net N$3: now also D2.P2K
- net N$5: now also D1.P2K
Other:
- moved on the sheet: D1, D3, X1-4
Changed lines of the file:
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@@
 <instance part="IC1" gate="D" x="142.24" y="38.1"/>
 <instance part="R4" gate="1" x="76.2" y="104.14" rot="R90"/>
-<instance part="D1" gate="G$1" x="76.2" y="93.98" rot="R270"/>
+<instance part="D1" gate="G$1" x="111.76" y="50.8" rot="R270"/>
 <instance part="U$34" gate="G$1" x="134.62" y="144.78" rot="R180"/>
 <instance part="U$35" gate="1" x="134.62" y="147.32" rot="R180"/>
@@
 <instance part="X1" gate="-2" x="53.34" y="60.96"/>
 <instance part="X1" gate="-3" x="73.66" y="40.64"/>
-<instance part="X1" gate="-4" x="43.18" y="154.94" rot="R180"/>
+<instance part="X1" gate="-4" x="101.6" y="129.54" rot="R180"/>
 <instance part="X1" gate="-5" x="91.44" y="129.54"/>
 <instance part="X1" gate="-6" x="213.36" y="76.2" rot="R180"/>
@@
 <instance part="X1" gate="-12" x="213.36" y="109.22" rot="R180"/>
 <instance part="D2" gate="G$1" x="91.44" y="71.12" rot="R270"/>
-<instance part="D3" gate="G$1" x="111.76" y="50.8" rot="R270"/>
+<instance part="D3" gate="G$1" x="76.2" y="93.98" rot="R270"/>
 <instance part="R5" gate="1" x="91.44" y="81.28" rot="R90"/>
 <instance part="U$37" gate="1" x="91.44" y="86.36" rot="R180"/>
@@
 <pinref part="X1" gate="-5" pin="1"/>
 <pinref part="U$32" gate="1" pin="GND"/>
+<pinref part="X1" gate="-4" pin="1"/>
+<junction x="96.52" y="129.54"/>
+<pinref part="X1" gate="-4" pin="1"/>
 </segment>
 <segment>
@@
 </segment>
 </net>
-<net name="N$18" class="0">
-<segment>
-<pinref part="D1" gate="G$1" pin="P1A"/>
-<pinref part="R4" gate="1" pin="1"/>
-</segment>
-</net>
 <net name="+5V" class="0">
 <segment>
@@
 <pinref part="D2" gate="G$1" pin="P1A"/>
 <pinref part="R5" gate="1" pin="1"/>
-</segment>
-</net>
-<net name="N$20" class="0">
-<segment>
-<pinref part="D3" gate="G$1" pin="P1A"/>
-<pinref part="R6" gate="1" pin="1"/>
 </segment>
 </net>
@@
 <pinref part="U$4" gate="G$1" pin="TP_13"/>
 <wire x1="127" y1="114.3" x2="73.66" y2="81.28" width="0.1524" layer="91"/>
+<wire x1="73.66" y1="81.28" x2="76.2" y2="86.36" width="0.1524" layer="91"/>
+<junction x="73.66" y="81.28"/>
+<pinref part="D3" gate="G$1" pin="P2K"/>
 </segment>
 </net>
@@
 <pinref part="U$5" gate="G$1" pin="TP_13"/>
 <wire x1="127" y1="109.22" x2="91.44" y2="60.96" width="0.1524" layer="91"/>
+<pinref part="D2" gate="G$1" pin="P2K"/>
+<wire x1="91.44" y1="60.96" x2="91.44" y2="63.5" width="0.1524" layer="91"/>
+<junction x="91.44" y="60.96"/>
 </segment>
 </net>
@@
 <pinref part="IC1" gate="C" pin="C"/>
 <pinref part="U$6" gate="G$1" pin="TP_13"/>
-<wire x1="127" y1="104.14" x2="111.76" y2="40.64" width="0.1524" layer="91"/>
-</segment>
-</net>
+<wire x1="127" y1="104.14" x2="111.76" y2="43.18" width="0.1524" layer="91"/>
+<pinref part="D1" gate="G$1" pin="P2K"/>
+<junction x="111.76" y="43.18"/>
+<wire x1="111.76" y1="43.18" x2="111.76" y2="40.64" width="0.1524" layer="91"/>
+</segment>
+</net>
+<net name="N$18" class="0">
+<segment>
+<pinref part="R4" gate="1" pin="1"/>
+<pinref part="D3" gate="G$1" pin="P1A"/>
+</segment>
+</net>
+<net name="N$20" class="0">
+<segment>
+<pinref part="R6" gate="1" pin="1"/>
+<pinref part="D1" gate="G$1" pin="P1A"/>
+</segment>
+</net>

Commit message: Arbeiten SW & SW zum 28.03.2020
Parts:
- removed U$10, U$21, U$9: LDD-H, SPEZIAL:LDD-H
- removed U$33: TP_10", SUPPLY:TP_10"
- added IC2, IC3: LDD-H, SPEZIAL:LDD-H
- added IC4: ILQ620, optocoupler:ILQ620
- added TESTPUNKT, U$39, U$40, U$41, U$42, U$43, U$44, U$45, U$46, U$47, U$48, U$49, U$50, U$51, U$52, U$53, U$54, U$55, U$56: TP_10", SUPPLY:TP_10"
- IC1: value ILQ620 -> LDD-H; device optocoupler:ILQ620 -> SPEZIAL:LDD-H
Connections:
- net N$18 renamed LED_3
- net N$19 renamed LED_2
- net N$20 renamed LED_1
- net SCHALTER_LI renamed SCHALTER_LI_1
- net SCHALTER_RE renamed SCHALTER_RE_1
- net SCHALTER_RUE renamed SCHALTER_RUE_1
- removed net N$1: IC1A.AC1, R1.2
- removed net N$10: U$10.-VOUT, X1-12.1
- removed net N$11: U$21.-VOUT, X1-7.1
- removed net N$12: U$21.+VOUT, X1-6.1
- removed net N$13: U$28.TP_13, U$9.DIMM
- removed net N$14: U$10.DIMM, U$29.TP_13
- removed net N$15: U$21.DIMM, U$30.TP_13
- removed net N$16: IC1D.C, U$3.TP_13
- removed net N$17: IC1D.AC1, U$33.TP_13
- removed net N$2: D3.P2K, IC1A.C, U$4.TP_13
- removed net N$3: D2.P2K, IC1B.C, U$5.TP_13
- removed net N$4: IC1B.AC1, R2.2
- removed net N$5: D1.P2K, IC1C.C, U$6.TP_13
- removed net N$6: IC1C.AC1, R3.2
- removed net N$7: U$9.+VOUT, X1-9.1
- removed net N$8: U$9.-VOUT, X1-10.1
- removed net N$9: U$10.+VOUT, X1-11.1
- new net +VOUT_1: IC1.+VOUT, X1-11.1
- new net +VOUT_2: IC2.+VOUT, X1-9.1
- new net +VOUT_3: IC3.+VOUT, X1-6.1
- new net -VOUT_1: IC1.-VOUT, X1-12.1
- new net -VOUT_2: IC2.-VOUT, X1-10.1
- new net -VOUT_3: IC3.-VOUT, X1-7.1
- new net DIMMER_1: IC1.DIMM, U$29.TP_13
- new net DIMMER_2: IC2.DIMM, U$28.TP_13
- new net DIMMER_3: IC3.DIMM, U$30.TP_13
- new net RESERVE_1: IC4D.AC1, TESTPUNKT.TP_13
- new net RESERVE_2: IC4D.C, U$3.TP_13
- new net SCH_LI_2: IC4B.AC1, R2.2
- new net SCH_LI_3: D2.P2K, IC4B.C, U$5.TP_13
- new net SCH_RE_2: IC4A.AC1, R1.2
- new net SCH_RE_3: D3.P2K, IC4A.C, U$4.TP_13
- new net SCH_RUE_2: IC4C.AC1, R3.2
- new net SCH_RUE_3: D1.P2K, IC4C.C, U$6.TP_13
- net +12V: now also IC1.+VIN, IC2.+VIN, IC3.+VIN; no longer U$10.+VIN, U$21.+VIN, U$9.+VIN
- net GND: now also IC1.-VIN, IC2.-VIN, IC3.-VIN, IC4A.AC2, IC4A.E, IC4B.AC2, IC4B.E, IC4C.AC2, IC4C.E, IC4D.AC2, IC4D.E; no longer IC1A.AC2, IC1A.E, IC1B.AC2, IC1B.E, IC1C.AC2, IC1C.E, IC1D.AC2, IC1D.E, U$10.-VIN, U$21.-VIN, U$9.-VIN
Other:
- moved on the sheet: D1, D2, D3, R1, R2, R3, R4, R5, R6, U$1, U$2, U$28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
