File: Eagle/Blinker_03.brd (EAGLE design)
At the start: 88.9 x 68.2 mm, 46 parts

Commit message: Cleanup
Routing:
- net N$3: track 0.00 -> 7.62 mm
- net N$4: track 0.00 -> 7.62 mm
- net N$2: track 0.00 -> 7.62 mm
- net N$5: track 0.00 -> 7.62 mm
Other:
- board size 88.9 x 68.2 mm -> 88.9 x 68.6 mm
- board text added: "BS"
- board text added: "LS"
Changed lines of the file:
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@@
 <plain>
 <wire x1="-8.89" y1="0" x2="79.99" y2="0" width="0" layer="20"/>
-<wire x1="79.99" y1="0" x2="79.99" y2="68.25" width="0" layer="20"/>
-<wire x1="79.99" y1="68.25" x2="-8.89" y2="68.25" width="0" layer="20"/>
-<wire x1="-8.89" y1="68.25" x2="-8.89" y2="0" width="0" layer="20"/>
+<wire x1="79.99" y1="0" x2="80.01" y2="68.58" width="0" layer="20"/>
+<wire x1="80.01" y1="68.58" x2="-8.89" y2="68.58" width="0" layer="20"/>
+<wire x1="-8.89" y1="68.58" x2="-8.89" y2="0" width="0" layer="20"/>
 <text x="45.085" y="38.1" size="1.778" layer="21">break</text>
 <text x="54.61" y="38.1" size="1.778" layer="21">left</text>
@@
 <rectangle x1="1.21328125" y1="50.83924375" x2="2.82364375" y2="50.92408125" layer="21" rot="R90"/>
 <rectangle x1="1.552753125" y1="50.415190625" x2="2.314753125" y2="50.499771875" layer="21" rot="R90"/>
+<text x="77.47" y="57.15" size="1.778" layer="16" rot="MR0">LS</text>
+<text x="73.66" y="57.15" size="1.778" layer="1">BS</text>
 </plain>
 <attributes>
@@
 <wire x1="36.83" y1="31.75" x2="36.83" y2="29.21" width="1.27" layer="16"/>
 <wire x1="59.69" y1="31.75" x2="59.69" y2="29.21" width="1.27" layer="16"/>
-<wire x1="-2.54" y1="46.99" x2="7.62" y2="46.99" width="1.27" layer="1"/>
-<wire x1="7.62" y1="46.99" x2="10.16" y2="49.53" width="1.27" layer="1"/>
-<wire x1="10.16" y1="49.53" x2="27.94" y2="49.53" width="1.27" layer="1"/>
+<wire x1="-2.54" y1="46.99" x2="7.62" y2="46.99" width="1.27" layer="16"/>
+<wire x1="7.62" y1="46.99" x2="10.16" y2="49.53" width="1.27" layer="16"/>
+<wire x1="10.16" y1="49.53" x2="27.94" y2="49.53" width="1.27" layer="16"/>
 <wire x1="13.97" y1="31.75" x2="13.97" y2="33.02" width="1.27" layer="16"/>
 <wire x1="13.97" y1="33.02" x2="15.24" y2="34.29" width="1.27" layer="16"/>
@@
 <wire x1="2.159" y1="26.67" x2="2.54" y2="27.051" width="1.27" layer="1"/>
 </signal>
+<signal name="N$2">
+<wire x1="80.01" y1="0" x2="80.01" y2="3.81" width="0.4064" layer="16"/>
+<wire x1="80.01" y1="0" x2="76.2" y2="0" width="0.4064" layer="16"/>
+</signal>
+<signal name="N$3">
+<wire x1="80.01" y1="68.58" x2="76.2" y2="68.58" width="0.4064" layer="16"/>
+<wire x1="80.01" y1="68.58" x2="80.01" y2="64.77" width="0.4064" layer="16"/>
+</signal>
+<signal name="N$4">
+<wire x1="-8.89" y1="68.58" x2="-5.08" y2="68.58" width="0.4064" layer="16"/>
+<wire x1="-8.89" y1="68.58" x2="-8.89" y2="64.77" width="0.4064" layer="16"/>
+</signal>
+<signal name="N$5">
+<wire x1="-8.89" y1="0" x2="-5.08" y2="0" width="0.4064" layer="16"/>
+<wire x1="-8.89" y1="0" x2="-8.89" y2="3.81" width="0.4064" layer="16"/>
+</signal>
 </signals>
