File: Eagle/Blinker_07.brd (EAGLE design)
At the start: 97.8 x 68.2 mm, 55 parts

Commit message: GY-61 Version 7.1
Parts:
- removed GND_GY-61, VCC-GY-61, X_OUT, Y_OUT, Z_OUT: TP_10", SUPPLY:TP_10
- added U1: GY-61, Indicator:GY-61
- moved R5 3.81 mm to (87.6, 29.2)
- moved S2 3.81 mm to (6.35, -7.62)
- moved OPTOKOPPLER 2.54 mm to (82.5, 12.7)
- moved U$46 2.54 mm to (91.4, 3.81)
- moved R2 2.54 mm to (87.6, 47.0)
- moved R6 2.54 mm to (87.6, 26.7)
- moved PLUG-2 1.27 mm to (97.8, 59.7)
- moved R1 1.27 mm to (87.6, 49.5)
- moved R3 1.27 mm to (87.6, 39.4)
Connections:
- removed net N$9: U$1.P$1, VCC-GY-61.P$1
- new net +3V3: U$1.P$1, U1.VDD
- net GND: now also U1.GND; no longer GND_GY-61.P$1
- net N$12: now also U1.X-OUT; no longer X_OUT.P$1
- net N$13: now also U1.Y-OUT; no longer Y_OUT.P$1
- net N$23: now also U1.Z-OUT; no longer Z_OUT.P$1
Routing:
- net +3V3: track 0.00 -> 50.1 mm, vias 0 -> 2
- net N$9: track 48.9 -> 0.00 mm, vias 2 -> 0
- net GND: track 287.7 -> 274.5 mm
- net +5V: track 61.8 -> 70.6 mm
- net N$20: track 21.9 -> 14.3 mm
- net N$24: track 32.8 -> 38.2 mm
- net INDICATOR-RIGHT: track 94.1 -> 97.9 mm
- net N$4: track 67.4 -> 71.0 mm
- net SCH_RE_3: track 71.2 -> 73.8 mm
- net BREAK: track 99.7 -> 102.2 mm
- net N$10: track 30.3 -> 32.8 mm
- net N$1: track 30.2 -> 32.8 mm
- net LED_2: track 35.7 -> 33.3 mm
- net N$2: track 8.15 -> 6.88 mm
- net N$11: track 16.3 -> 15.0 mm
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Other:
- board size 97.8 x 68.2 mm -> 99 x 68.6 mm
- board text added: "COPS SHOULD NOT READ THIS"
- board text added: "Fuze:"
- board text added: "Made by : S.W & S.W Date : 05/10/2020"
