File: Eagle/Blinker_07.brd (EAGLE design)
At the start: 99 x 68.6 mm, 51 parts, among them U1 GY-61

Commit message: 7.2 Mutter freigelegt
Parts:
- removed S1, S2: TL32PO, switch:TL3XPO
- moved R5 6.35 mm to (87.6, 27.9)
- moved R1 3.81 mm to (87.6, 53.3)
- moved R2 3.81 mm to (87.6, 50.8)
- moved R3 3.81 mm to (87.6, 48.3)
- moved U1 2.54 mm to (77.5, 38.1)
- moved PLUG-2 1.27 mm to (97.8, 61.0)
- moved R4 1.27 mm to (87.6, 38.1)
- moved R6 1.27 mm to (87.6, 25.4)
Routing:
- net N$1: track 32.8 -> 24.4 mm
- net INDICATOR-RIGHT: track 92.8 -> 99.2 mm
- net GND: track 292.5 -> 286.5 mm
- net N$11: track 18.6 -> 13.8 mm
- net +3V3: track 47.6 -> 50.1 mm
- net LED_2: track 28.2 -> 30.6 mm
- net +5V: track 67.4 -> 69.7 mm
- net N$24: track 37.4 -> 38.7 mm
- net N$22: track 18.3 -> 17.0 mm
- net BREAK: track 102.2 -> 103.5 mm
- net N$2: track 6.88 -> 7.40 mm
- net N$20: track 14.3 -> 14.8 mm
- net INDICATOR-LEFT: track 88.5 -> 87.9 mm

Commit message: 7.2 Fehlerbehebung
Routing:
- net BREAK: track 103.5 -> 104.2 mm
- net INDICATOR-LEFT: track 87.9 -> 87.2 mm
Changed lines of the file:
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@@
 <element name="U$1" library="SUPPLY" package="TP_10" value="TP_10&quot;" x="55.88" y="7.62"/>
 <element name="U1" library="Indicator" package="GY-61" value="GY-61" x="77.47" y="38.1" smashed="yes" rot="R180">
-<attribute name="NAME" x="81.28" y="38.1" size="1.27" layer="25" rot="R180"/>
+<attribute name="NAME" x="81.28" y="33.02" size="1.27" layer="25" rot="R180"/>
 <attribute name="VALUE" x="78.74" y="34.29" size="1.27" layer="27"/>
 </element>
@@
 <wire x1="55.88" y1="38.1" x2="64.77" y2="38.1" width="1.4224" layer="1"/>
 <wire x1="86.36" y1="58.42" x2="86.36" y2="45.72" width="1.4224" layer="16"/>
-<wire x1="86.36" y1="43.18" x2="86.36" y2="25.4" width="1.4224" layer="16"/>
+<wire x1="86.36" y1="45.72" x2="86.36" y2="25.4" width="1.4224" layer="16"/>
 <wire x1="86.36" y1="25.4" x2="82.55" y2="21.59" width="1.4224" layer="16"/>
 <wire x1="77.47" y1="43.18" x2="83.82" y2="43.18" width="1.4224" layer="16"/>
 <wire x1="83.82" y1="43.18" x2="86.36" y2="45.72" width="1.4224" layer="16"/>
-<wire x1="86.36" y1="45.72" x2="86.36" y2="43.18" width="1.4224" layer="16"/>
 <wire x1="64.77" y1="38.1" x2="69.85" y2="43.18" width="1.4224" layer="16"/>
 <wire x1="69.85" y1="43.18" x2="73.66" y2="43.18" width="1.4224" layer="16"/>
@@
 <contactref element="R4" pad="1"/>
 <contactref element="PLUG-12" pad="5"/>
-<wire x1="82.55" y1="38.1" x2="81.28" y2="38.1" width="0.4064" layer="1"/>
-<wire x1="81.28" y1="38.1" x2="81.28" y2="45.72" width="0.4064" layer="1"/>
-<wire x1="81.28" y1="45.72" x2="80.01" y2="46.99" width="0.4064" layer="1"/>
+<wire x1="82.55" y1="38.1" x2="82.55" y2="44.45" width="0.4064" layer="1"/>
+<wire x1="82.55" y1="44.45" x2="80.01" y2="46.99" width="0.4064" layer="1"/>
 <wire x1="80.01" y1="46.99" x2="10.16" y2="46.99" width="0.4064" layer="1"/>
 <wire x1="10.16" y1="46.99" x2="8.89" y2="45.72" width="0.4064" layer="1"/>
@@
 <wire x1="10.16" y1="44.45" x2="11.43" y2="45.72" width="0.4064" layer="1"/>
 <wire x1="11.43" y1="45.72" x2="78.74" y2="45.72" width="0.4064" layer="1"/>
-<wire x1="78.74" y1="45.72" x2="80.01" y2="44.45" width="0.4064" layer="1"/>
-<wire x1="80.01" y1="44.45" x2="80.01" y2="30.48" width="0.4064" layer="1"/>
-<wire x1="80.01" y1="30.48" x2="82.55" y2="27.94" width="0.4064" layer="1"/>
+<wire x1="78.74" y1="45.72" x2="81.28" y2="43.18" width="0.4064" layer="1"/>
+<wire x1="81.28" y1="43.18" x2="81.28" y2="29.21" width="0.4064" layer="1"/>
+<wire x1="81.28" y1="29.21" x2="82.55" y2="27.94" width="0.4064" layer="1"/>
 </signal>
 <signal name="BREAK">
@@
 <wire x1="11.43" y1="33.02" x2="11.43" y2="43.18" width="0.4064" layer="1"/>
 <wire x1="11.43" y1="43.18" x2="12.7" y2="44.45" width="0.4064" layer="1"/>
-<wire x1="12.7" y1="44.45" x2="77.47" y2="44.45" width="0.4064" layer="1"/>
-<wire x1="77.47" y1="44.45" x2="78.74" y2="43.18" width="0.4064" layer="1"/>
-<wire x1="78.74" y1="43.18" x2="78.74" y2="29.21" width="0.4064" layer="1"/>
-<wire x1="78.74" y1="29.21" x2="82.55" y2="25.4" width="0.4064" layer="1"/>
+<wire x1="12.7" y1="44.45" x2="78.74" y2="44.45" width="0.4064" layer="1"/>
+<wire x1="78.74" y1="44.45" x2="80.01" y2="43.18" width="0.4064" layer="1"/>
+<wire x1="80.01" y1="43.18" x2="80.01" y2="27.94" width="0.4064" layer="1"/>
+<wire x1="80.01" y1="27.94" x2="82.55" y2="25.4" width="0.4064" layer="1"/>
 </signal>
 <signal name="BLUE-LED">

Commit message: 7.2 große löcher
Routing:
- net INDICATOR-LEFT: track 87.2 -> 86.5 mm
Changed lines of the file:
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@@
 <setting verticaltext="up"/>
 </settings>
-<grid distance="50" unitdist="mil" unit="mil" style="lines" multiple="1" display="yes" altdistance="0.025" altunitdist="inch" altunit="inch"/>
+<grid distance="50" unitdist="mil" unit="mm" style="lines" multiple="1" display="yes" altdistance="0.025" altunitdist="inch" altunit="inch"/>
 <layers>
 <layer number="1" name="Top" color="4" fill="1" visible="yes" active="yes"/>
@@
 <contactref element="R4" pad="1"/>
 <contactref element="PLUG-12" pad="5"/>
-<wire x1="82.55" y1="38.1" x2="82.55" y2="44.45" width="0.4064" layer="1"/>
-<wire x1="82.55" y1="44.45" x2="80.01" y2="46.99" width="0.4064" layer="1"/>
-<wire x1="80.01" y1="46.99" x2="10.16" y2="46.99" width="0.4064" layer="1"/>
+<wire x1="82.55" y1="38.1" x2="82.55" y2="43.18" width="0.4064" layer="1"/>
+<wire x1="82.55" y1="43.18" x2="78.74" y2="46.99" width="0.4064" layer="1"/>
+<wire x1="78.74" y1="46.99" x2="10.16" y2="46.99" width="0.4064" layer="1"/>
 <wire x1="10.16" y1="46.99" x2="8.89" y2="45.72" width="0.4064" layer="1"/>
 <wire x1="8.89" y1="45.72" x2="8.89" y2="43.18" width="0.4064" layer="1"/>
