File: Eagle/Blinker_07.sch (EAGLE design)
At the start: 51 parts

Commit message: GY-61 Version 7.1
Parts:
- removed U$5: TP_10", SUPPLY:TP_10"
- added U1: GY-61, Indicator:GY-61
Connections:
- new net +3V3: U$1.TP_13, U1.VDD
- new net N$12: U$56.TP_13, U1.X-OUT
- new net N$13: U$49.TP_13, U1.Y-OUT
- new net N$23: U$48.TP_13, U1.Z-OUT
- net GND: now also U1.GND; no longer U$5.TP_13
Other:
- moved on the sheet: OPTOKOPPLERC, PLUG-12-8, U$1, U$45, U$48, U$49, U$56
Changed lines of the file:
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@@
 <setting verticaltext="up"/>
 </settings>
-<grid distance="0.1" unitdist="inch" unit="inch" style="lines" multiple="1" display="no" altdistance="0.01" altunitdist="inch" altunit="inch"/>
+<grid distance="0.05" unitdist="inch" unit="inch" style="lines" multiple="1" display="no" altdistance="0.01" altunitdist="inch" altunit="inch"/>
 <layers>
 <layer number="1" name="Top" color="4" fill="1" visible="no" active="no"/>
@@
 <part name="S2" library="switch" deviceset="TL32PO" device=""/>
 <part name="U$1" library="SUPPLY" deviceset="TP_10" device="&quot;"/>
-<part name="U$5" library="SUPPLY" deviceset="TP_10" device="&quot;"/>
+<part name="U$5" library="SUPPLY" deviceset="GND" device=""/>
+<part name="+3V1" library="supply1" deviceset="+3V3" device=""/>
+<part name="+3V2" library="supply1" deviceset="+3V3" device=""/>
+<part name="U1" library="Indicator" deviceset="GY-61" device=""/>
 </parts>
 <sheets>
@@
 <wire x1="137.16" y1="76.2" x2="137.16" y2="165.1" width="0.1524" layer="94"/>
 <wire x1="281.94" y1="12.7" x2="256.54" y2="12.7" width="0.1524" layer="94"/>
-<wire x1="281.94" y1="81.28" x2="281.94" y2="12.7" width="0.1524" layer="94"/>
-<wire x1="256.54" y1="81.28" x2="256.54" y2="12.7" width="0.1524" layer="94"/>
-<wire x1="281.94" y1="81.28" x2="256.54" y2="81.28" width="0.1524" layer="94"/>
+<wire x1="281.94" y1="63.5" x2="281.94" y2="12.7" width="0.1524" layer="94"/>
+<wire x1="256.54" y1="63.5" x2="256.54" y2="12.7" width="0.1524" layer="94"/>
+<wire x1="281.94" y1="63.5" x2="256.54" y2="63.5" width="0.1524" layer="94"/>
 </plain>
 <instances>
@@
 <attribute name="VALUE" x="84.455" y="154.94" size="1.778" layer="96"/>
 </instance>
-<instance part="OPTOKOPPLER" gate="C" x="91.44" y="76.2" smashed="yes">
-<attribute name="NAME" x="79.375" y="81.915" size="1.778" layer="95"/>
-<attribute name="VALUE" x="84.455" y="68.58" size="1.778" layer="96"/>
+<instance part="OPTOKOPPLER" gate="C" x="88.9" y="76.2" smashed="yes">
+<attribute name="NAME" x="76.835" y="81.915" size="1.778" layer="95"/>
+<attribute name="VALUE" x="81.915" y="68.58" size="1.778" layer="96"/>
 </instance>
 <instance part="OPTOKOPPLER" gate="D" x="91.44" y="121.92" smashed="yes">
@@
 <instance part="PLUG-12" gate="-6" x="60.96" y="124.46"/>
 <instance part="PLUG-12" gate="-7" x="60.96" y="78.74"/>
-<instance part="PLUG-12" gate="-8" x="271.78" y="119.38" rot="R90"/>
+<instance part="PLUG-12" gate="-8" x="269.24" y="124.46" rot="R270"/>
 <instance part="PLUG-12" gate="-9" x="233.68" y="129.54" rot="R180"/>
 <instance part="PLUG-12" gate="-10" x="233.68" y="124.46" rot="R180"/>
@@
 <instance part="U$43" gate="G$1" x="279.4" y="53.34" rot="R90"/>
 <instance part="U$44" gate="G$1" x="279.4" y="60.96" rot="R90"/>
-<instance part="U$45" gate="G$1" x="279.4" y="68.58" rot="R90"/>
+<instance part="U$45" gate="G$1" x="259.08" y="60.96" rot="R270"/>
 <instance part="U$46" gate="G$1" x="76.2" y="35.56" rot="R90"/>
 <instance part="U$47" gate="G$1" x="175.26" y="101.6" rot="R90"/>
-<instance part="U$48" gate="G$1" x="259.08" y="76.2" rot="R270"/>
-<instance part="U$49" gate="G$1" x="259.08" y="68.58" rot="R270"/>
+<instance part="U$48" gate="G$1" x="171.45" y="78.74"/>
+<instance part="U$49" gate="G$1" x="166.37" y="78.74"/>
 <instance part="U$50" gate="G$1" x="259.08" y="15.24" rot="R270"/>
 <instance part="U$51" gate="G$1" x="259.08" y="22.86" rot="R270"/>
@@
 <instance part="U$54" gate="G$1" x="259.08" y="45.72" rot="R270"/>
 <instance part="U$55" gate="G$1" x="259.08" y="53.34" rot="R270"/>
-<instance part="U$56" gate="G$1" x="259.08" y="60.96" rot="R270"/>
+<instance part="U$56" gate="G$1" x="161.29" y="78.74"/>
 <instance part="F1" gate="G$1" x="30.48" y="172.72" rot="R180"/>
 <instance part="R1" gate="1" x="106.68" y="142.24" rot="R90"/>
@@
 <instance part="S1" gate="BEF1" x="27.94" y="22.86" rot="R270"/>
 <instance part="S2" gate="BEF1" x="17.78" y="22.86" rot="R270"/>
-<instance part="U$1" gate="G$1" x="279.4" y="76.2" rot="R90"/>
-<instance part="U$5" gate="G$1" x="157.48" y="132.08" rot="R270"/>
+<instance part="U$1" gate="G$1" x="142.24" y="81.28" rot="R270"/>
+<instance part="U$5" gate="1" x="130.81" y="53.34"/>
+<instance part="+3V1" gate="G$1" x="129.54" y="83.82"/>
+<instance part="+3V2" gate="G$1" x="130.81" y="62.23"/>
+<instance part="U1" gate="G$1" x="142.24" y="55.88"/>
 </instances>
 <busses>
@@
 <segment>
 <pinref part="U$18" gate="1" pin="GND"/>
-<wire x1="132.08" y1="127" x2="132.08" y2="132.08" width="0.1524" layer="91"/>
 <pinref part="GND_2" gate="G$1" pin="TP_13"/>
-<wire x1="154.94" y1="132.08" x2="132.08" y2="132.08" width="0.1524" layer="91"/>
-<wire x1="132.08" y1="132.08" x2="132.08" y2="137.16" width="0.1524" layer="91"/>
+<wire x1="132.08" y1="127" x2="132.08" y2="137.16" width="0.1524" layer="91"/>
 <wire x1="132.08" y1="137.16" x2="139.7" y2="137.16" width="0.1524" layer="91"/>
 <pinref part="GND_1" gate="G$1" pin="TP_13"/>
 <wire x1="139.7" y1="127" x2="132.08" y2="127" width="0.1524" layer="91"/>
 <junction x="132.08" y="127"/>
-<pinref part="U$5" gate="G$1" pin="TP_13"/>
-<junction x="154.94" y="132.08"/>
 </segment>
 <segment>
@@
 <pinref part="OPTOKOPPLER" gate="C" pin="E"/>
 <pinref part="U$15" gate="1" pin="GND"/>
-<wire x1="106.68" y1="73.66" x2="104.14" y2="73.66" width="0.1524" layer="91"/>
+<wire x1="106.68" y1="73.66" x2="101.6" y2="73.66" width="0.1524" layer="91"/>
 </segment>
 <segment>
 <pinref part="OPTOKOPPLER" gate="C" pin="AC2"/>
 <pinref part="U$16" gate="1" pin="GND"/>
-<wire x1="78.74" y1="73.66" x2="81.28" y2="73.66" width="0.1524" layer="91"/>
 </segment>
 <segment>
@@
 <wire x1="20.32" y1="160.02" x2="30.48" y2="160.02" width="0.1524" layer="91"/>
 </segment>
+<segment>
+<pinref part="U$5" gate="1" pin="GND"/>
+<pinref part="U1" gate="G$1" pin="GND"/>
+<wire x1="130.81" y1="53.34" x2="133.35" y2="53.34" width="0.1524" layer="91"/>
+</segment>
 </net>
 <net name="+12V" class="0">
@@
 <wire x1="119.38" y1="111.76" x2="119.38" y2="165.1" width="0.1524" layer="91"/>
 <pinref part="OPTOKOPPLER" gate="B" pin="C"/>
-<wire x1="119.38" y1="165.1" x2="104.14" y2="165.1" width="0.1524" layer="91"/>
-<junction x="119.38" y="165.1"/>
+<wire x1="119.38" y1="165.1" x2="106.68" y2="165.1" width="0.1524" layer="91"/>
 <pinref part="D1" gate="G$1" pin="P2K"/>
-<junction x="104.14" y="165.1"/>
 <wire x1="104.14" y1="165.1" x2="106.68" y2="165.1" width="0.1524" layer="91"/>
 <pinref part="A4" gate="G$1" pin="TP_13"/>
+<junction x="106.68" y="165.1"/>
 </segment>
 </net>
@@
 <wire x1="114.3" y1="96.52" x2="114.3" y2="78.74" width="0.1524" layer="91"/>
 <pinref part="OPTOKOPPLER" gate="C" pin="C"/>
-<wire x1="114.3" y1="78.74" x2="104.14" y2="78.74" width="0.1524" layer="91"/>
+<wire x1="114.3" y1="78.74" x2="106.68" y2="78.74" width="0.1524" layer="91"/>
 <pinref part="D2" gate="G$1" pin="P2K"/>
-<junction x="104.14" y="78.74"/>
-<wire x1="104.14" y1="78.74" x2="106.68" y2="78.74" width="0.1524" layer="91"/>
+<wire x1="101.6" y1="78.74" x2="106.68" y2="78.74" width="0.1524" layer="91"/>
 <pinref part="A3" gate="G$1" pin="TP_13"/>
+<junction x="106.68" y="78.74"/>
 </segment>
 </net>
@@
 <pinref part="OPTOKOPPLER" gate="C" pin="AC1"/>
 <pinref part="R6" gate="1" pin="2"/>
-<wire x1="78.74" y1="78.74" x2="81.28" y2="78.74" width="0.1524" layer="91"/>
 </segment>
 </net>
@@
 </segment>
 </net>
+<net name="N$12" class="0">
+<segment>
+<pinref part="U$56" gate="G$1" pin="TP_13"/>
+<wire x1="161.29" y1="76.2" x2="161.29" y2="60.96" width="0.1524" layer="91"/>
+<pinref part="U1" gate="G$1" pin="X-OUT"/>
+<wire x1="161.29" y1="60.96" x2="156.21" y2="60.96" width="0.1524" layer="91"/>
+</segment>
+</net>
+<net name="N$13" class="0">
+<segment>
+<pinref part="U$49" gate="G$1" pin="TP_13"/>
+<wire x1="166.37" y1="76.2" x2="166.37" y2="55.88" width="0.1524" layer="91"/>
+<pinref part="U1" gate="G$1" pin="Y-OUT"/>
+<wire x1="166.37" y1="55.88" x2="156.21" y2="55.88" width="0.1524" layer="91"/>
+</segment>
+</net>
+<net name="N$23" class="0">
+<segment>
+<pinref part="U$48" gate="G$1" pin="TP_13"/>
+<pinref part="U1" gate="G$1" pin="Z-OUT"/>
+<wire x1="156.21" y1="50.8" x2="171.45" y2="50.8" width="0.1524" layer="91"/>
+<wire x1="171.45" y1="50.8" x2="171.45" y2="76.2" width="0.1524" layer="91"/>
+</segment>
+</net>
+<net name="+3V3" class="0">
+<segment>
+<pinref part="+3V2" gate="G$1" pin="+3V3"/>
+<wire x1="130.81" y1="59.69" x2="130.81" y2="58.42" width="0.1524" layer="91"/>
+<pinref part="U1" gate="G$1" pin="VDD"/>
+<wire x1="130.81" y1="58.42" x2="133.35" y2="58.42" width="0.1524" layer="91"/>
+</segment>
+<segment>
+<pinref part="U$1" gate="G$1" pin="TP_13"/>
+<pinref part="+3V1" gate="G$1" pin="+3V3"/>
+<wire x1="129.54" y1="81.28" x2="139.7" y2="81.28" width="0.1524" layer="91"/>
+</segment>
+</net>

Commit message: 7.2 Mutter freigelegt
Parts:
- removed S1, S2: TL32PO, switch:TL32PO
Changed lines of the file:
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@@
 <setting verticaltext="up"/>
 </settings>
-<grid distance="0.05" unitdist="inch" unit="inch" style="lines" multiple="1" display="no" altdistance="0.01" altunitdist="inch" altunit="inch"/>
+<grid distance="0.1" unitdist="inch" unit="inch" style="lines" multiple="1" display="no" altdistance="0.01" altunitdist="inch" altunit="inch"/>
 <layers>
 <layer number="1" name="Top" color="4" fill="1" visible="no" active="no"/>
@@
 <part name="U$4" library="SUPPLY" deviceset="GND" device=""/>
 <part name="PLUG-2" library="con-phoenix-508" deviceset="MSTBA2" device=""/>
-<part name="S1" library="switch" deviceset="TL32PO" device=""/>
-<part name="S2" library="switch" deviceset="TL32PO" device=""/>
 <part name="U$1" library="SUPPLY" deviceset="TP_10" device="&quot;"/>
 <part name="U$5" library="SUPPLY" deviceset="GND" device=""/>
@@
 <instance part="PLUG-2" gate="-1" x="15.24" y="160.02"/>
 <instance part="PLUG-2" gate="-2" x="15.24" y="172.72"/>
-<instance part="S1" gate="BEF1" x="27.94" y="22.86" rot="R270"/>
-<instance part="S2" gate="BEF1" x="17.78" y="22.86" rot="R270"/>
 <instance part="U$1" gate="G$1" x="142.24" y="81.28" rot="R270"/>
 <instance part="U$5" gate="1" x="130.81" y="53.34"/>

Commit message: 7.2 große löcher
Changed lines of the file:
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@@
 <instance part="+3V1" gate="G$1" x="129.54" y="83.82"/>
 <instance part="+3V2" gate="G$1" x="130.81" y="62.23"/>
-<instance part="U1" gate="G$1" x="142.24" y="55.88"/>
+<instance part="U1" gate="G$1" x="144.78" y="55.88"/>
 </instances>
 <busses>
@@
 <pinref part="U$5" gate="1" pin="GND"/>
 <pinref part="U1" gate="G$1" pin="GND"/>
-<wire x1="130.81" y1="53.34" x2="133.35" y2="53.34" width="0.1524" layer="91"/>
+<wire x1="130.81" y1="53.34" x2="134.62" y2="53.34" width="0.1524" layer="91"/>
 </segment>
 </net>
@@
 <wire x1="161.29" y1="76.2" x2="161.29" y2="60.96" width="0.1524" layer="91"/>
 <pinref part="U1" gate="G$1" pin="X-OUT"/>
-<wire x1="161.29" y1="60.96" x2="156.21" y2="60.96" width="0.1524" layer="91"/>
+<wire x1="161.29" y1="60.96" x2="160.02" y2="60.96" width="0.1524" layer="91"/>
 </segment>
 </net>
@@
 <wire x1="166.37" y1="76.2" x2="166.37" y2="55.88" width="0.1524" layer="91"/>
 <pinref part="U1" gate="G$1" pin="Y-OUT"/>
-<wire x1="166.37" y1="55.88" x2="156.21" y2="55.88" width="0.1524" layer="91"/>
+<wire x1="166.37" y1="55.88" x2="160.02" y2="55.88" width="0.1524" layer="91"/>
 </segment>
 </net>
@@
 <pinref part="U$48" gate="G$1" pin="TP_13"/>
 <pinref part="U1" gate="G$1" pin="Z-OUT"/>
-<wire x1="156.21" y1="50.8" x2="171.45" y2="50.8" width="0.1524" layer="91"/>
+<wire x1="160.02" y1="50.8" x2="171.45" y2="50.8" width="0.1524" layer="91"/>
 <wire x1="171.45" y1="50.8" x2="171.45" y2="76.2" width="0.1524" layer="91"/>
 </segment>
@@
 <wire x1="130.81" y1="59.69" x2="130.81" y2="58.42" width="0.1524" layer="91"/>
 <pinref part="U1" gate="G$1" pin="VDD"/>
-<wire x1="130.81" y1="58.42" x2="133.35" y2="58.42" width="0.1524" layer="91"/>
-</segment>
-<segment>
+<wire x1="130.81" y1="58.42" x2="134.62" y2="58.42" width="0.1524" layer="91"/>
+</segment>
+<segment>
