File: Eagle/Layout für PCB-Pool/Blink.brd (EAGLE design)
At the start: 133.3 x 68.6 mm, 80 parts, among them IC1 78L05, IC2 MAX3232CPE, IC3 MAX3232CPE, IC4 78L05

Commit message: SWE: Nutzen für PCB-Pool
Parts:
- C1, C2: value (none) -> 1µ; device R-C:C050-025X075 -> R-C:ES-2,5L
- C3, C4: value 1µ -> 10µ
- C5, C6: value 10µ -> (none); device R-C:ES-2,5L -> R-C:C050-025X075
- moved C101 25.4 mm to (132.7, 43.8)
- moved C102 25.4 mm to (132.7, 51.4)
- moved C103 25.4 mm to (120.0, 56.5)
- moved C104 25.4 mm to (132.7, 59.1)
- moved C4 21.9 mm to (109.9, 59.1)
- moved C3 21.1 mm to (109.9, 38.1)
- moved C6 14.4 mm to (120.0, 47.6), turned to 270 degrees
- moved C1 13.6 mm to (109.9, 45.1), turned to 90 degrees
- moved C2 8.08 mm to (109.9, 52.1), turned to 90 degrees
- moved C5 4.96 mm to (126.4, 40.0), turned to 180 degrees
- moved IC4 4.62 mm to (118.7, 40.0)
- moved IC3 4.62 mm to (126.4, 52.7)
- moved U$8 3.42 mm to (130.2, 16.5)
- moved U$9 3.42 mm to (130.2, 25.4)
- moved 8 3.42 mm to (127.6, 34.9)
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Connections:
- removed net N$3: C3.1, IC3.1
- removed net N$4: C3.2, IC3.3
- removed net N$5: C4.1, IC3.4
- removed net N$6: C4.2, IC3.5
- new net N$10: C101.1, IC3.3
- new net N$11: C102.2, IC3.4
- new net N$12: C102.1, IC3.5
- new net N$13: C103.1, IC3.2
- new net N$14: C104.1, IC3.6
- new net N$16: X1.7, X1.8
- new net N$17: X1.1, X1.4, X1.6
- new net N$9: C101.2, IC3.1
- net +5V1: now also C3.2; no longer C103.2
- net +5V2: now also C103.2, C6.2; no longer C2.2, C5.2
- net CABLE_PIN_1: now also C5.2; no longer C1.2
- net GND1: now also C4.1; no longer C104.2
- net GND2: now also C104.2, C5.1; no longer C1.1, C2.1
- net N$21: now also C1.1; no longer C101.2
- net N$22: now also C1.2; no longer C101.1
- net N$23: now also C2.1; no longer C102.2
- net N$24: now also C2.2; no longer C102.1
- net N$25: now also C3.1; no longer C103.1
- net N$26: now also C4.2; no longer C104.1
- net N$7: now also X2.7, X2.8; no longer C5.1, IC3.2
- net N$8: now also X2.1, X2.4, X2.6; no longer C6.2, IC3.6
Routing:
- net N$15: track 0.00 -> 21.6 mm
- net N$13: track 0.00 -> 20.6 mm
- net N$17: track 0.00 -> 20.0 mm, vias 0 -> 2
- net N$2: track 21.6 -> 7.62 mm
- net N$26: track 2.54 -> 11.5 mm
- net N$16: track 0.00 -> 8.84 mm
- net N$8: track 11.5 -> 19.3 mm, vias 0 -> 2
- net N$7: track 15.0 -> 8.90 mm
- net N$25: track 20.6 -> 15.0 mm
- net N$11: track 0.00 -> 4.34 mm
- net N$10: track 0.00 -> 3.59 mm
- net +5V1: track 19.4 -> 22.4 mm
- net +5V2: track 22.4 -> 19.4 mm
- net GND2: track 66.3 -> 63.3 mm
- net GND1: track 63.3 -> 66.3 mm
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Other:
- board size 133.3 x 68.6 mm -> 135.9 x 68.6 mm
- board text added: "BS"
- board text added: "LS"
